Commit message: world map transform in tams setup urdf file
Before this change we had to publish an static transform via a command line.

File: tams_ur5_setup_description/urdf/tams_ur5_setup.urdf.xacro (robot description, xacro)
@@ -13,4 +13,10 @@
     <origin xyz="0.0 0.0 0.0" rpy="0.0 0.0 0.0" />
   </joint>
+  <link name="map" />
+  <joint name="map_world" type="fixed">
+    <parent link="world" />
+    <child link = "map" />
+    <origin xyz="0.9 1.3 0.0" rpy="0.0 0.0 -0.32" />
+  </joint>
   <joint name="wall_ur5_joint" type="fixed">
     <parent link="wall" />

Commit message: Set prefix for ur5 arm
We want to insert a new link tool0 as eef for the arm at the origin of
the fts_toolside. The ur5 already has a tool0 at another position, so we
set a prefix.

For more information see the commit:
1c08ba42b1087d9042ebe69f1e1033736084145a

File: tams_ur5_setup_description/urdf/tams_ur5_setup.urdf.xacro (robot description, xacro)
@@ -21,5 +21,5 @@
   <joint name="wall_ur5_joint" type="fixed">
     <parent link="wall" />
-    <child link = "base_link" />
+    <child link = "ur5_base_link" />
     <origin xyz="0.0 0.722 1.0175" rpy="${pi/2} 0.0 ${pi/2}" />
   </joint>
