Commit message: Apriltag rotation in urdf
moved apriltag rotation from the camera_positioner to the urdf file of
the TAMS laboratory corner
added pi as constant to urdf file

File: tams_ur5_setup_description/urdf/tams_corner.urdf.xacro (robot description, xacro)
@@ -3,4 +3,5 @@
        name="tams_corner" >
   <xacro:property name="roomheight" value="3.0" />
+  <xacro:property name="pi" value="3.1415926535897931" />
   <material name="white">
     <color rgba="1 1 1 1"/>
@@ -202,5 +203,5 @@
       <origin xyz="0 0 0" />
       <geometry>
-        <box size="0.01 0.166 0.166" />
+        <box size="0.166 0.166 0.01" />
       </geometry>
     </visual>
@@ -208,5 +209,5 @@
       <origin xyz="0 0 0.0" />
       <geometry>
-        <box size="0.01 0.166 0.166" />
+        <box size="0.166 0.166 0.01" />
       </geometry>
     </collision>
@@ -256,5 +257,5 @@
     <child link = "april_tag_ur5" />
     <!--<origin xyz="0.06 -1.75 -0.23" rpy="0.0 0.0 0.0" />-->
-    <origin xyz="-0.01 0.75 1.27" rpy="0.0 0.0 0.0" /> <!-- offset relative to the tilted wall -->
+    <origin xyz="-0.01 0.75 1.27" rpy="${pi/2} 0.0 ${pi/2}" /> <!-- offset relative to the tilted wall -->
   </joint>
 </robot>

Commit message: Add cable-duct to tams_corner urdf and moveit collisions

File: tams_ur5_setup_description/urdf/tams_corner.urdf.xacro (robot description, xacro)
@@ -133,4 +133,34 @@
     <kd>1.0</kd>
   </gazebo>
+  <link name="cable_duct">
+    <inertial>
+      <origin xyz="0 0 0" />
+      <mass value="2000" />
+      <inertia  ixx="1" ixy="0" ixz="0" iyy="1" iyz="0" izz="1" />
+    </inertial>
+    <visual>
+      <material name="lightgray" />
+      <origin xyz="0 0 0" />
+      <geometry>
+        <box size="0.13 0.08 ${roomheight}" />
+      </geometry>
+    </visual>
+    <collision>
+      <origin xyz="0 0 0.0" />
+      <geometry>
+        <box size="0.13 0.08 ${roomheight}" />
+      </geometry>
+    </collision>
+  </link>
+  <gazebo reference="cable_duct">
+    <material>Gazebo/Blue</material>
+    <turnGravityOff>false</turnGravityOff>
+    <selfCollide>true</selfCollide>
+    <!-- kp: stiffness kd: damping mu1, mu2: friction -->
+    <mu1>100.0</mu1>
+    <mu2>100.0</mu2>
+    <kp>1000000.0</kp>
+    <kd>1.0</kd>
+  </gazebo>
   <link name="table">
     <inertial>
@@ -239,5 +269,10 @@
     <child link="small_wall"/>
     <!--<origin xyz="2.5 -0.06 1.5" rpy="0 0 0" />-->
-    <origin xyz="0.095 -0.0825 1.5" rpy="0 0 0" />
+    <origin xyz="0.07 -0.0825 1.5" rpy="0 0 0" />
+  </joint>
+  <joint name="cable_duct_joint" type="fixed">
+    <parent link="floor"/>
+    <child link="cable_duct"/>
+    <origin xyz="0.375 -0.125 ${roomheight/2}" rpy="0 0 0" />
   </joint>
   <joint name="table_joint" type="fixed">

Commit message: resized visual model for cabel duct
visual model from 8cm to 6cm reduced.
Collision model still 8cm because of an ethernet port.

File: tams_ur5_setup_description/urdf/tams_corner.urdf.xacro (robot description, xacro)
@@ -143,10 +143,11 @@
       <origin xyz="0 0 0" />
       <geometry>
-        <box size="0.13 0.08 ${roomheight}" />
-      </geometry>
-    </visual>
-    <collision>
-      <origin xyz="0 0 0.0" />
-      <geometry>
+        <box size="0.13 0.06 ${roomheight}" />
+      </geometry>
+    </visual>
+    <collision>
+      <origin xyz="0 0 0" />
+      <geometry>
+        <!-- the collision model is 2cm wider then the actual duct, because of an unmodelled ethernet port -->
         <box size="0.13 0.08 ${roomheight}" />
       </geometry>
@@ -274,5 +275,5 @@
     <parent link="floor"/>
     <child link="cable_duct"/>
-    <origin xyz="0.375 -0.125 ${roomheight/2}" rpy="0 0 0" />
+    <origin xyz="0.375 -0.135 ${roomheight/2}" rpy="0 0 0" />
   </joint>
   <joint name="table_joint" type="fixed">

Commit message: corrected error of measurement of cable duct
cable duct is shiftet by 47,5 cm instead of 37,5 cm in x direction

File: tams_ur5_setup_description/urdf/tams_corner.urdf.xacro (robot description, xacro)
@@ -275,5 +275,5 @@
     <parent link="floor"/>
     <child link="cable_duct"/>
-    <origin xyz="0.375 -0.135 ${roomheight/2}" rpy="0 0 0" />
+    <origin xyz="0.475 -0.135 ${roomheight/2}" rpy="0 0 0" />
   </joint>
   <joint name="table_joint" type="fixed">

Commit message: Fill gap between floor and side wall in tams corner urdf
Due to the modeling of the cable duct and the small wall the position of
the side wall was moved. The outcome of this was a small gap between the
wall and the floor.

File: tams_ur5_setup_description/urdf/tams_corner.urdf.xacro (robot description, xacro)
@@ -23,5 +23,5 @@
       <origin xyz="2.5 2.5 0" />
       <geometry>
-        <box size="5.0 5.0 0.001" />
+        <box size="5.0 5.33 0.001" />
       </geometry>
     </visual>
@@ -29,5 +29,5 @@
       <origin xyz="2.5 2.5 0" />
       <geometry>
-      <box size="5.0 5.0 0.001" />
+      <box size="5.0 5.33 0.001" />
       </geometry>
     </collision>

Commit message: Correctly increased just one side of the floor from the last commit

File: tams_ur5_setup_description/urdf/tams_corner.urdf.xacro (robot description, xacro)
@@ -21,13 +21,13 @@
     <visual>
       <material name="black" />
-      <origin xyz="2.5 2.5 0" />
-      <geometry>
-        <box size="5.0 5.33 0.001" />
-      </geometry>
-    </visual>
-    <collision>
-      <origin xyz="2.5 2.5 0" />
-      <geometry>
-      <box size="5.0 5.33 0.001" />
+      <origin xyz="2.5 2.4175 0" />
+      <geometry>
+        <box size="5.0 5.165 0.001" />
+      </geometry>
+    </visual>
+    <collision>
+      <origin xyz="2.5 2.4175 0" />
+      <geometry>
+      <box size="5.0 5.165 0.001" />
       </geometry>
     </collision>

Commit message: New table with different size in the laboratory
Changed the size of the table in the urdf file to the values of the new table

File: tams_ur5_setup_description/urdf/tams_corner.urdf.xacro (robot description, xacro)
@@ -166,5 +166,5 @@
   <link name="table">
     <inertial>
-      <origin xyz="0 0 0.365" />
+      <origin xyz="0 0 0.37" />
       <mass value="10" />
       <inertia  ixx="1" ixy="0" ixz="0" iyy="1" iyz="0" izz="1" />
@@ -172,13 +172,13 @@
     <visual>
       <material name="brown" />
-      <origin xyz="0 0 0.365" />
-      <geometry>
-        <box size="0.67 0.67 0.73" />
-      </geometry>
-    </visual>
-    <collision>
-      <origin xyz="0 0 0.365" />
-      <geometry>
-        <box size="0.67 0.67 0.73" />
+      <origin xyz="0 0 0.37" />
+      <geometry>
+        <box size="1.0 0.80 0.74" />
+      </geometry>
+    </visual>
+    <collision>
+      <origin xyz="0 0 0.37" />
+      <geometry>
+        <box size="1.0 0.80 0.74" />
       </geometry>
     </collision>
@@ -281,5 +281,5 @@
     <child link="table"/>
     <!-- actual wall is 2.5cm further back from table, but is modelled at the position of the small ur5 adapter plate -->
-    <origin xyz="0.58 0.23 0" rpy="0 0 0" />
+    <origin xyz="0.73 0.30 0" rpy="0 0 0" />
   </joint>
   <joint name="shelf_joint" type="fixed">

Commit message: New link table_top
New link in the middle of the table surface. This link is inserted link
the object from it, instead of the world frame.

With this link we could visualize the object always from the surface of
the table.

File: tams_ur5_setup_description/urdf/tams_corner.urdf.xacro (robot description, xacro)
@@ -4,4 +4,5 @@
   <xacro:property name="roomheight" value="3.0" />
   <xacro:property name="pi" value="3.1415926535897931" />
+  <xacro:property name="tableheight" value="0.74" />
   <material name="white">
     <color rgba="1 1 1 1"/>
@@ -166,5 +167,5 @@
   <link name="table">
     <inertial>
-      <origin xyz="0 0 0.37" />
+      <origin xyz="0 0 ${tableheight/2}" />
       <mass value="10" />
       <inertia  ixx="1" ixy="0" ixz="0" iyy="1" iyz="0" izz="1" />
@@ -172,13 +173,13 @@
     <visual>
       <material name="brown" />
-      <origin xyz="0 0 0.37" />
-      <geometry>
-        <box size="1.0 0.80 0.74" />
-      </geometry>
-    </visual>
-    <collision>
-      <origin xyz="0 0 0.37" />
-      <geometry>
-        <box size="1.0 0.80 0.74" />
+      <origin xyz="0 0 ${tableheight/2}" />
+      <geometry>
+        <box size="1.0 0.80 ${tableheight}" />
+      </geometry>
+    </visual>
+    <collision>
+      <origin xyz="0 0 ${tableheight/2}" />
+      <geometry>
+        <box size="1.0 0.80 ${tableheight}" />
       </geometry>
     </collision>
@@ -194,4 +195,5 @@
     <kd>1.0</kd>
   </gazebo>
+  <link name="table_top"/>
   <link name="shelf">
     <inertial>
@@ -282,4 +284,9 @@
     <!-- actual wall is 2.5cm further back from table, but is modelled at the position of the small ur5 adapter plate -->
     <origin xyz="0.73 0.30 0" rpy="0 0 0" />
+  </joint>
+  <joint name="table_top_joint" type="fixed">
+    <parent link="table"/>
+    <child link="table_top"/>
+    <origin xyz="0 0 ${tableheight}" rpy="0 0 0"/>
   </joint>
   <joint name="shelf_joint" type="fixed">

Commit message: Change position of apriltag 0
the tag 0 is moved to a position over the metal plate and is glued on a
piece of wood. Now the camera detect the apriltag more solid.

File: tams_ur5_setup_description/urdf/tams_corner.urdf.xacro (robot description, xacro)
@@ -299,6 +299,5 @@
     <parent link="wall" />
     <child link = "april_tag_ur5" />
-    <!--<origin xyz="0.06 -1.75 -0.23" rpy="0.0 0.0 0.0" />-->
-    <origin xyz="-0.01 0.75 1.27" rpy="${pi/2} 0.0 ${pi/2}" /> <!-- offset relative to the tilted wall -->
+    <origin xyz="-0.02 0.75 1.494" rpy="${-pi/2} 0.0 ${-pi/2}" /> <!-- offset relative to the tilted wall -->
   </joint>
 </robot>

Commit message: links turtlebot and turtlebot_holder
Two new links were established in the urdf.
One for the turtlebot and one for the holder on the top of the
turtlebot. Due to this, we can reference the poses for placing the
object to this frames.

File: tams_ur5_setup_description/urdf/tams_corner.urdf.xacro (robot description, xacro)
@@ -255,4 +255,6 @@
     <kd>1.0</kd>
   </gazebo>
+  <link name="turtlebot" />
+  <link name="turtlebot_holder" />
   <joint name="floor_wall_joint" type="fixed">
     <parent link="floor"/>
@@ -296,8 +298,18 @@
     <origin xyz="0.2 1 1.25" rpy="0 0 0" />
   </joint>
-   <joint name="apriltag_ur5_joint" type="fixed">
+  <joint name="apriltag_ur5_joint" type="fixed">
     <parent link="wall" />
-    <child link = "april_tag_ur5" />
+    <child link="april_tag_ur5" />
     <origin xyz="-0.02 0.75 1.494" rpy="${-pi/2} 0.0 ${-pi/2}" /> <!-- offset relative to the tilted wall -->
   </joint>
+  <joint name="turtlebot_joint" type="fixed">
+    <parent link="world" />
+    <child link="turtlebot" />
+    <origin xyz="0.26 1.31 0.0" rpy="0.0 0.0 0.0" />
+  </joint>
+  <joint name="turtlebot_holder_joint" type="fixed">
+    <parent link="turtlebot" />
+    <child link="turtlebot_holder" />
+    <origin xyz="0.035 0.0 0.42" rpy="0.0 0.0 0.0" />
+  </joint>
 </robot>

Commit message: Corrected values for turtlebot_holder frame

File: tams_ur5_setup_description/urdf/tams_corner.urdf.xacro (robot description, xacro)
@@ -311,5 +311,5 @@
     <parent link="turtlebot" />
     <child link="turtlebot_holder" />
-    <origin xyz="0.035 0.0 0.42" rpy="0.0 0.0 0.0" />
+    <origin xyz="0.04 0.0 0.41" rpy="0.0 0.0 0.0" />
   </joint>
 </robot>

Commit message: Increase collision boxes for cable duct and small wall
The robot often moves very close to the cabke duct and the small wall in
the corner. So we increased the collision model that the planner will
find a plan with more distence.

File: tams_ur5_setup_description/urdf/tams_corner.urdf.xacro (robot description, xacro)
@@ -114,5 +114,5 @@
       <origin xyz="0 0 0" />
       <geometry>
-        <box size="0.19 0.165 3.0" />
+              <box size="0.19 0.165 ${roomheight}" />
       </geometry>
     </visual>
@@ -120,5 +120,6 @@
       <origin xyz="0 0 0.0" />
       <geometry>
-        <box size="0.19 0.165 3.0" />
+        <!-- the collision model is 7cm wider due to security reasons -->
+        <box size="0.33 0.305 ${roomheight}" />
       </geometry>
     </collision>
@@ -150,6 +151,6 @@
       <origin xyz="0 0 0" />
       <geometry>
-        <!-- the collision model is 2cm wider then the actual duct, because of an unmodelled ethernet port -->
-        <box size="0.13 0.08 ${roomheight}" />
+        <!-- the collision model is 7cm wider then the actual duct, because of an unmodelled ethernet port -->
+        <box size="0.27 0.2 ${roomheight}" />
       </geometry>
     </collision>

Commit message: Increase of shelf collision model size

File: tams_ur5_setup_description/urdf/tams_corner.urdf.xacro (robot description, xacro)
@@ -213,5 +213,6 @@
       <origin xyz="0 1.7 0" />
       <geometry>
-        <box size="0.4 2 2.5" />
+        <!-- the collision model is 7cm wider due to security reasons -->
+        <box size="0.54 2.14 2.5" />
       </geometry>
     </collision>

Commit message: refine corner model

File: tams_ur5_setup_description/urdf/tams_corner.urdf.xacro (robot description, xacro)
@@ -303,5 +303,5 @@
     <parent link="wall" />
     <child link="april_tag_ur5" />
-    <origin xyz="-0.02 0.75 1.494" rpy="${-pi/2} 0.0 ${-pi/2}" /> <!-- offset relative to the tilted wall -->
+    <origin xyz="-0.015 0.75 1.494" rpy="${-pi/2} 0.0 ${-pi/2}" /> <!-- offset relative to the tilted wall -->
   </joint>
   <joint name="turtlebot_joint" type="fixed">

Commit message: project2016 setup. * changing table position. * adding named target definition.

File: tams_ur5_setup_description/urdf/tams_corner.urdf.xacro (robot description, xacro)
@@ -4,5 +4,5 @@
   <xacro:property name="roomheight" value="3.0" />
   <xacro:property name="pi" value="3.1415926535897931" />
-  <xacro:property name="tableheight" value="0.74" />
+  <xacro:property name="tableheight" value="0.75" />
   <material name="white">
     <color rgba="1 1 1 1"/>
@@ -172,9 +172,9 @@
       <inertia  ixx="1" ixy="0" ixz="0" iyy="1" iyz="0" izz="1" />
     </inertial>
-    <visual>
+   <visual>
       <material name="brown" />
       <origin xyz="0 0 ${tableheight/2}" />
       <geometry>
-        <box size="1.0 0.80 ${tableheight}" />
+        <box size="0.80 1.0 ${tableheight}" />
       </geometry>
     </visual>
@@ -182,9 +182,9 @@
       <origin xyz="0 0 ${tableheight/2}" />
       <geometry>
-        <box size="1.0 0.80 ${tableheight}" />
-      </geometry>
-    </collision>
-  </link>
-  <gazebo reference="table">
+        <box size="0.80 1.0 ${tableheight}" />
+      </geometry>
+    </collision>
+</link>
+<gazebo reference="table">
     <material>Gazebo/Blue</material>
     <turnGravityOff>false</turnGravityOff>
@@ -264,5 +264,5 @@
     <!-- The actual wall in the lab is slightly tilted, the rotation compensates approx 1 deg -->
     <origin xyz="0 0 0" rpy="0 0 0" />
-    <!--<origin xyz="0 0 0" rpy="0 -0.017 0" />-->
+    <!--<origin xyz="0 0 0" rpy="0 0.06 0" />-->
   </joint>
   <joint name="side_wall_joint" type="fixed">
@@ -287,5 +287,6 @@
     <child link="table"/>
     <!-- actual wall is 2.5cm further back from table, but is modelled at the position of the small ur5 adapter plate -->
-    <origin xyz="0.73 0.30 0" rpy="0 0 0" />
+   <!-- <origin xyz="0.75 0.3 0" rpy="0 0 0" /> -->
+    <origin xyz="0.89 0.74 0" rpy="0 0 0" />
   </joint>
   <joint name="table_top_joint" type="fixed">
@@ -303,4 +304,5 @@
     <parent link="wall" />
     <child link="april_tag_ur5" />
+    <!--<origin xyz="-0.015 0.75 1.494" rpy="${-pi/2-0.05} 0.0 ${-pi/2}" />--> <!-- offset relative to the tilted wall -->
     <origin xyz="-0.015 0.75 1.494" rpy="${-pi/2} 0.0 ${-pi/2}" /> <!-- offset relative to the tilted wall -->
   </joint>

Commit message: Add ur5 wall mount description and adjust kinematic chain

File: tams_ur5_setup_description/urdf/tams_corner.urdf.xacro (robot description, xacro)
@@ -74,4 +74,20 @@
     <kd>1.0</kd>
   </gazebo>
+  <!-- tilted ur5 mount - the meshes are not centered at mount point so they are adjusted to fit to the frame -->
+  <link name="ur5_mount">
+    <visual>
+      <material name="lightgray" />
+      <origin xyz="-0.0245 -0.09 -0.28" />
+      <geometry>
+	<mesh filename="package://tams_ur5_setup_description/meshes/ur5_mount_binary_v3.stl" scale="0.001 0.001 0.001"/>
+      </geometry>
+    </visual>
+    <collision>
+      <origin xyz="-0.0245 -0.09 -0.28" />
+      <geometry>
+	<mesh filename="package://tams_ur5_setup_description/meshes/ur5_mount_binary_v3.stl" scale="0.001 0.001 0.001"/>
+      </geometry>
+    </collision>
+  </link>
   <link name="side_wall">
     <inertial>
@@ -265,4 +281,9 @@
     <origin xyz="0 0 0" rpy="0 0 0" />
     <!--<origin xyz="0 0 0" rpy="0 -0.017 0" />-->
+  </joint>
+  <joint name="wall_mount_joint" type="fixed">
+    <parent link="wall"/>
+    <child link="ur5_mount"/>
+	<origin xyz="0.2255 0.7245 1.085" rpy="0 0 ${pi}" />
   </joint>
   <joint name="side_wall_joint" type="fixed">

Commit message: Adds tilted wall mount description and attaches arm to it.

File: tams_ur5_setup_description/urdf/tams_corner.urdf.xacro (robot description, xacro)
@@ -74,4 +74,20 @@
     <kd>1.0</kd>
   </gazebo>
+  <!-- tilted ur5 mount - the meshes are not centered at mount point so they are adjusted to fit to the frame -->
+  <link name="ur5_mount">
+    <visual>
+      <material name="lightgray" />
+      <origin xyz="-0.0245 -0.09 -0.28" />
+      <geometry>
+	<mesh filename="package://tams_ur5_setup_description/meshes/ur5_mount_binary_v3.stl" scale="0.001 0.001 0.001"/>
+      </geometry>
+    </visual>
+    <collision>
+      <origin xyz="-0.0245 -0.09 -0.28" />
+      <geometry>
+	<mesh filename="package://tams_ur5_setup_description/meshes/ur5_mount_binary_v3.stl" scale="0.001 0.001 0.001"/>
+      </geometry>
+    </collision>
+  </link>
   <link name="side_wall">
     <inertial>
@@ -265,4 +281,9 @@
     <origin xyz="0 0 0" rpy="0 0 0" />
     <!--<origin xyz="0 0 0" rpy="0 0.06 0" />-->
+  </joint>
+  <joint name="wall_mount_joint" type="fixed">
+    <parent link="wall"/>
+    <child link="ur5_mount"/>
+	<origin xyz="0.2255 0.7245 1.085" rpy="0 0 ${pi}" />
   </joint>
   <joint name="side_wall_joint" type="fixed">

File: tams_ur5_setup_description/urdf/tams_ur5_setup.urdf.xacro (robot description, xacro)
@@ -20,7 +20,7 @@
   </joint>
   <joint name="wall_ur5_joint" type="fixed">
-    <parent link="wall" />
+    <parent link="ur5_mount" />
     <child link = "ur5_base_link" />
-    <origin xyz="0.0 0.722 1.0175" rpy="${pi/2} 0.0 ${pi/2}" />
+    <origin xyz="0 0 0.003" rpy="0.0 0.0 ${pi/2}" />
   </joint>
 </robot>

Commit message: Adding clock collision object. Adjusting april tag position.

File: tams_ur5_setup_description/urdf/tams_corner.urdf.xacro (robot description, xacro)
@@ -251,5 +251,5 @@
     </inertial>
     <visual>
-      <material name="black" />
+      <material name="lightgray" />
       <origin xyz="0 0 0" />
       <geometry>
@@ -273,4 +273,24 @@
     <kd>1.0</kd>
   </gazebo>
+  <link name="clock">
+    <inertial>
+      <origin xyz="0 0 0" />
+      <mass value="2000" />
+      <inertia  ixx="1" ixy="0" ixz="0" iyy="1" iyz="0" izz="1" />
+    </inertial>
+    <visual>
+      <material name="lightgray" />
+      <origin xyz="0 0 0" />
+      <geometry>
+        <cylinder length="0.06" radius="0.14"/>
+      </geometry>
+    </visual>
+    <collision>
+      <origin xyz="0 0 0.0" />
+      <geometry>
+        <cylinder length="0.06" radius="0.14"/>
+      </geometry>
+    </collision>
+  </link>
   <link name="turtlebot" />
   <link name="turtlebot_holder" />
@@ -326,5 +346,10 @@
     <child link="april_tag_ur5" />
     <!--<origin xyz="-0.015 0.75 1.494" rpy="${-pi/2-0.05} 0.0 ${-pi/2}" />--> <!-- offset relative to the tilted wall -->
-    <origin xyz="-0.015 0.75 1.494" rpy="${-pi/2} 0.0 ${-pi/2}" /> <!-- offset relative to the tilted wall -->
+    <origin xyz="-0.01 0.75 1.494" rpy="${-pi/2} 0.0 ${-pi/2}" /> <!-- offset relative to the tilted wall -->
+  </joint>
+  <joint name="clock_joint" type="fixed">
+    <parent link="wall" />
+    <child link="clock" />
+    <origin xyz="0.03 0.82 1.993" rpy="${-pi/2} 0.0 ${-pi/2}" /> <!-- offset relative to the tilted wall -->
   </joint>
   <joint name="turtlebot_joint" type="fixed">

Commit message: Fix clock height

File: tams_ur5_setup_description/urdf/tams_corner.urdf.xacro (robot description, xacro)
@@ -351,5 +351,5 @@
     <parent link="wall" />
     <child link="clock" />
-    <origin xyz="0.03 0.82 1.993" rpy="${-pi/2} 0.0 ${-pi/2}" /> <!-- offset relative to the tilted wall -->
+    <origin xyz="0.03 0.82 1.93" rpy="${-pi/2} 0.0 ${-pi/2}" /> <!-- offset relative to the tilted wall -->
   </joint>
   <joint name="turtlebot_joint" type="fixed">

Commit message: Fix april tag position

File: tams_ur5_setup_description/urdf/tams_corner.urdf.xacro (robot description, xacro)
@@ -305,5 +305,5 @@
     <parent link="wall"/>
     <child link="ur5_mount"/>
-	<origin xyz="0.2255 0.7245 1.085" rpy="0 0 ${pi}" />
+	<origin xyz="0.2255 0.7245 1.082" rpy="0 0 ${pi}" />
   </joint>
   <joint name="side_wall_joint" type="fixed">
@@ -346,5 +346,5 @@
     <child link="april_tag_ur5" />
     <!--<origin xyz="-0.015 0.75 1.494" rpy="${-pi/2-0.05} 0.0 ${-pi/2}" />--> <!-- offset relative to the tilted wall -->
-    <origin xyz="-0.01 0.75 1.494" rpy="${-pi/2} 0.0 ${-pi/2}" /> <!-- offset relative to the tilted wall -->
+    <origin xyz="-0.01 0.74 1.505" rpy="${-pi/2} 0.0 ${-pi/2}" /> <!-- offset relative to the tilted wall -->
   </joint>
   <joint name="clock_joint" type="fixed">

Commit message: Change table height

File: tams_ur5_setup_description/urdf/tams_corner.urdf.xacro (robot description, xacro)
@@ -4,5 +4,5 @@
   <xacro:property name="roomheight" value="3.0" />
   <xacro:property name="pi" value="3.1415926535897931" />
-  <xacro:property name="tableheight" value="0.74" />
+  <xacro:property name="tableheight" value="0.75" />
   <material name="white">
     <color rgba="1 1 1 1"/>
