Commit message: Rotate table and fix april tag position

File: tams_ur5_setup_description/urdf/tams_corner.urdf.xacro (robot description, xacro)
@@ -176,5 +176,5 @@
       <origin xyz="0 0 ${tableheight/2}" />
       <geometry>
-        <box size="1.0 0.80 ${tableheight}" />
+        <box size="0.80 1.0 ${tableheight}" />
       </geometry>
     </visual>
@@ -182,5 +182,5 @@
       <origin xyz="0 0 ${tableheight/2}" />
       <geometry>
-        <box size="1.0 0.80 ${tableheight}" />
+        <box size="0.80 1.0 ${tableheight}" />
       </geometry>
     </collision>
@@ -287,5 +287,6 @@
     <child link="table"/>
     <!-- actual wall is 2.5cm further back from table, but is modelled at the position of the small ur5 adapter plate -->
-    <origin xyz="0.73 0.30 0" rpy="0 0 0" />
+   <!-- <origin xyz="0.73 0.30 0" rpy="0 0 0" /> -->
+    <origin xyz="0.89 0.74 0" rpy="0 0 0" />
   </joint>
   <joint name="table_top_joint" type="fixed">
@@ -303,4 +304,5 @@
     <parent link="wall" />
     <child link="april_tag_ur5" />
+    <!-- <origin xyz="-0.015 0.75 1.494" rpy="${-pi/2-0.05} 0.0 ${-pi/2}" /> --> <!-- with rotation correction -->
     <origin xyz="-0.015 0.75 1.494" rpy="${-pi/2} 0.0 ${-pi/2}" /> <!-- offset relative to the tilted wall -->
   </joint>

Commit message: Add clock collision object and adjust april tag position

File: tams_ur5_setup_description/urdf/tams_corner.urdf.xacro (robot description, xacro)
@@ -251,5 +251,5 @@
     </inertial>
     <visual>
-      <material name="black" />
+      <material name="lightgray" />
       <origin xyz="0 0 0" />
       <geometry>
@@ -273,4 +273,24 @@
     <kd>1.0</kd>
   </gazebo>
+  <link name="clock">
+    <inertial>
+      <origin xyz="0 0 0" />
+      <mass value="2000" />
+      <inertia  ixx="1" ixy="0" ixz="0" iyy="1" iyz="0" izz="1" />
+    </inertial>
+    <visual>
+      <material name="lightgray" />
+      <origin xyz="0 0 0" />
+      <geometry>
+        <cylinder length="0.06" radius="0.14"/>
+      </geometry>
+    </visual>
+    <collision>
+      <origin xyz="0 0 0.0" />
+      <geometry>
+        <cylinder length="0.06" radius="0.14"/>
+      </geometry>
+    </collision>
+  </link>
   <link name="turtlebot" />
   <link name="turtlebot_holder" />
@@ -326,5 +346,10 @@
     <child link="april_tag_ur5" />
     <!-- <origin xyz="-0.015 0.75 1.494" rpy="${-pi/2-0.05} 0.0 ${-pi/2}" /> --> <!-- with rotation correction -->
-    <origin xyz="-0.015 0.75 1.494" rpy="${-pi/2} 0.0 ${-pi/2}" /> <!-- offset relative to the tilted wall -->
+    <origin xyz="-0.01 0.75 1.494" rpy="${-pi/2} 0.0 ${-pi/2}" /> <!-- offset relative to the tilted wall -->
+  </joint>
+  <joint name="clock_joint" type="fixed">
+    <parent link="wall" />
+    <child link="clock" />
+    <origin xyz="0.03 0.82 1.993" rpy="${-pi/2} 0.0 ${-pi/2}" /> <!-- offset relative to the tilted wall -->
   </joint>
   <joint name="turtlebot_joint" type="fixed">

Commit message: Fix positions of april tag and ur5 mount

File: tams_ur5_setup_description/urdf/tams_corner.urdf.xacro (robot description, xacro)
@@ -305,5 +305,5 @@
     <parent link="wall"/>
     <child link="ur5_mount"/>
-	<origin xyz="0.2255 0.7245 1.085" rpy="0 0 ${pi}" />
+	<origin xyz="0.2255 0.7245 1.082" rpy="0 0 ${pi}" />
   </joint>
   <joint name="side_wall_joint" type="fixed">
@@ -346,5 +346,5 @@
     <child link="april_tag_ur5" />
     <!-- <origin xyz="-0.015 0.75 1.494" rpy="${-pi/2-0.05} 0.0 ${-pi/2}" /> --> <!-- with rotation correction -->
-    <origin xyz="-0.01 0.75 1.494" rpy="${-pi/2} 0.0 ${-pi/2}" /> <!-- offset relative to the tilted wall -->
+    <origin xyz="-0.01 0.74 1.505" rpy="${-pi/2} 0.0 ${-pi/2}" /> <!-- offset relative to the tilted wall -->
   </joint>
   <joint name="clock_joint" type="fixed">

Commit message: Fine adjust april tag position and size

File: tams_ur5_setup_description/urdf/tams_corner.urdf.xacro (robot description, xacro)
@@ -346,5 +346,5 @@
     <child link="april_tag_ur5" />
     <!-- <origin xyz="-0.015 0.75 1.494" rpy="${-pi/2-0.05} 0.0 ${-pi/2}" /> --> <!-- with rotation correction -->
-    <origin xyz="-0.01 0.74 1.505" rpy="${-pi/2} 0.0 ${-pi/2}" /> <!-- offset relative to the tilted wall -->
+    <origin xyz="-0.009 0.74 1.505" rpy="${-pi/2} 0.0 ${-pi/2+0.015}" /> <!-- offset relative to the tilted wall -->
   </joint>
   <joint name="clock_joint" type="fixed">

Commit message: Implement optional floating table
The table of the setup can move.
If we track the april tags on the table and the wall,
we can publish the transform online and don't have to
rely on the static transform. MoveIt will extract the
joint state from TF.

File: tams_ur5_setup_description/urdf/tams_corner.urdf.xacro (robot description, xacro)
@@ -2,7 +2,11 @@
 <robot xmlns:xacro="http://www.ros.org/wiki/xacro"
        name="tams_corner" >
+  <xacro:arg name="floating_table" default="false" />
   <xacro:property name="roomheight" value="3.0" />
   <xacro:property name="pi" value="3.1415926535897931" />
   <xacro:property name="tableheight" value="0.75" />
+  <xacro:property name="tablewidth" value="1.00" />
+  <xacro:property name="tabledepth" value="0.80" />
+  <xacro:property name="tabletag_size" value="0.20" />
   <material name="white">
     <color rgba="1 1 1 1"/>
@@ -213,4 +217,5 @@
   </gazebo>
   <link name="table_top"/>
+  <link name="table_tag"/>
   <link name="shelf">
     <inertial>
@@ -324,4 +329,5 @@
     <origin xyz="0.475 -0.135 ${roomheight/2}" rpy="0 0 0" />
   </joint>
+  <xacro:unless value="$(arg floating_table)">
   <joint name="table_joint" type="fixed">
     <parent link="floor"/>
@@ -331,8 +337,20 @@
     <origin xyz="0.89 0.74 0" rpy="0 0 0" />
   </joint>
+  </xacro:unless>
+  <xacro:if value="$(arg floating_table)">
+  <joint name="table_joint" type="floating">
+    <parent link="floor"/>
+    <child link="table"/>
+  </joint>
+  </xacro:if>
   <joint name="table_top_joint" type="fixed">
     <parent link="table"/>
     <child link="table_top"/>
     <origin xyz="0 0 ${tableheight}" rpy="0 0 0"/>
+  </joint>
+  <joint name="table_tag_joint" type="fixed">
+    <parent link="table_top"/>
+    <child link="table_tag"/>
+    <origin xyz="${tabledepth/2-tabletag_size/2} ${tablewidth/2-tabletag_size/2} 0" rpy="0 0 0"/>
   </joint>
   <joint name="shelf_joint" type="fixed">

File: tams_ur5_setup_description/urdf/tams_ur5_setup.urdf.xacro (robot description, xacro)
@@ -4,5 +4,7 @@
   <xacro:property name="pi" value="3.1415926535897931" />
   <!-- tams corner -->
-  <xacro:include filename="$(find tams_ur5_setup_description)/urdf/tams_corner.urdf.xacro" />
+  <xacro:include filename="$(find tams_ur5_setup_description)/urdf/tams_corner.urdf.xacro">
+    <arg name="floating_table" value="$(arg floating_table)" />
+  </xacro:include>
   <!-- arm -->
   <xacro:include filename="$(find tams_ur5_description)/urdf/arm.urdf.xacro" />

Commit message: someone... glued the tag onto the table the wrong way around...
Most likely that someone was me... sorry.

File: tams_ur5_setup_description/urdf/tams_corner.urdf.xacro (robot description, xacro)
@@ -352,5 +352,5 @@
     <parent link="table_top"/>
     <child link="table_tag"/>
-    <origin xyz="${tabledepth/2-tabletag_size/2} ${tablewidth/2-tabletag_size/2} 0" rpy="0 0 0"/>
+    <origin xyz="${tabledepth/2-tabletag_size/2} ${tablewidth/2-tabletag_size/2} 0" rpy="0 0 ${pi}"/>
   </joint>
   <joint name="shelf_joint" type="fixed">

Commit message: Update table height to 78cm

File: tams_ur5_setup_description/urdf/tams_corner.urdf.xacro (robot description, xacro)
@@ -5,5 +5,5 @@
   <xacro:property name="roomheight" value="3.0" />
   <xacro:property name="pi" value="3.1415926535897931" />
-  <xacro:property name="tableheight" value="0.75" />
+  <xacro:property name="tableheight" value="0.78" />
   <xacro:property name="tablewidth" value="1.00" />
   <xacro:property name="tabledepth" value="0.80" />

Commit message: Add ur5_mount_plate as parent link of ur5_mount

File: tams_ur5_setup_description/urdf/tams_corner.urdf.xacro (robot description, xacro)
@@ -78,4 +78,6 @@
     <kd>1.0</kd>
   </gazebo>
+  <!-- frame of the ur5 mount plate -->
+  <link name="ur5_mount_plate"/>
   <!-- tilted ur5 mount - the meshes are not centered at mount point so they are adjusted to fit to the frame -->
   <link name="ur5_mount">
@@ -307,8 +309,13 @@
     <!--<origin xyz="0 0 0" rpy="0 -0.017 0" />-->
   </joint>
+  <joint name="wall_mount_plate_joint" type="fixed">
+    <parent link="wall"/>
+    <child link="ur5_mount_plate"/>
+	<origin xyz="0.0 0.7245 1.05" rpy="0 0 0" />
+  </joint>
   <joint name="wall_mount_joint" type="fixed">
-    <parent link="wall"/>
+    <parent link="ur5_mount_plate"/>
     <child link="ur5_mount"/>
-	<origin xyz="0.2255 0.7245 1.082" rpy="0 0 ${pi}" />
+	<origin xyz="0.2255 -0.025 0.032" rpy="0 0 ${pi}" />
   </joint>
   <joint name="side_wall_joint" type="fixed">

Commit message: remove definition of pi as it already predefined

File: tams_ur5_setup_description/urdf/tams_corner.urdf.xacro (robot description, xacro)
@@ -4,5 +4,4 @@
   <xacro:arg name="floating_table" default="false" />
   <xacro:property name="roomheight" value="3.0" />
-  <xacro:property name="pi" value="3.1415926535897931" />
   <xacro:property name="tableheight" value="0.78" />
   <xacro:property name="tablewidth" value="1.00" />

File: tams_ur5_setup_description/urdf/tams_ur5_setup.urdf.xacro (robot description, xacro)
@@ -2,5 +2,4 @@
 <robot xmlns:xacro="http://www.ros.org/wiki/xacro"
        name="tams_ur5_setup" >
-  <xacro:property name="pi" value="3.1415926535897931" />
   <!-- tams corner -->
   <xacro:include filename="$(find tams_ur5_setup_description)/urdf/tams_corner.urdf.xacro">

Commit message: remove deprecated plugin

File: tams_ur5_setup_description/urdf/tams_corner.urdf.xacro (robot description, xacro)
@@ -8,4 +8,7 @@
   <xacro:property name="tabledepth" value="0.80" />
   <xacro:property name="tabletag_size" value="0.20" />
+  <material name="black">
+    <color rgba="0.0 0.0 0.0 1.0"/>
+  </material>
   <material name="white">
     <color rgba="1 1 1 1"/>

Commit message: make corner-walls transparent
to finally get rid of most camera angles not showing the actual robot.

File: tams_ur5_setup_description/urdf/tams_corner.urdf.xacro (robot description, xacro)
@@ -57,5 +57,7 @@
     </inertial>
     <visual>
-      <material name="white" />
+      <material name="wall_mat">
+        <color rgba="1.0 1.0 1.0 0.4" />
+      </material>
       <origin xyz="-0.06 2.5 1.5" />
       <geometry>
@@ -105,5 +107,7 @@
     </inertial>
     <visual>
-      <material name="white" />
+      <material name="side_wall_mat">
+        <color rgba="1.0 1.0 1.0 0.4" />
+      </material>
       <origin xyz="0 0 0" />
       <geometry>
@@ -135,5 +139,7 @@
     </inertial>
     <visual>
-      <material name="white" />
+      <material name="small_wall_mat">
+        <color rgba="1.0 1.0 1.0 0.4" />
+      </material>
       <origin xyz="0 0 0" />
       <geometry>
@@ -166,5 +172,7 @@
     </inertial>
     <visual>
-      <material name="lightgray" />
+      <material name="cable_duct_mat">
+        <color rgba="0.7 0.7 0.7 0.4" />
+      </material>
       <origin xyz="0 0 0" />
       <geometry>
@@ -229,5 +237,7 @@
     </inertial>
     <visual>
-      <material name="lightgray" />
+      <material name="shelf_mat">
+        <color rgba="0.7 0.7 0.7 0.4" />
+      </material>
       <origin xyz="0 1.7 0" />
       <geometry>
@@ -289,5 +299,7 @@
     </inertial>
     <visual>
-      <material name="lightgray" />
+      <material name="clock_mat">
+        <color rgba="0.7 0.7 0.7 0.4" />
+      </material>
       <origin xyz="0 0 0" />
       <geometry>

Commit message: move table to top level file as it is optional
... as discussed with Norman

File: tams_ur5_setup_description/urdf/tams_corner.urdf.xacro (robot description, xacro)
@@ -2,10 +2,5 @@
 <robot xmlns:xacro="http://www.ros.org/wiki/xacro"
        name="tams_corner" >
-  <xacro:arg name="floating_table" default="false" />
   <xacro:property name="roomheight" value="3.0" />
-  <xacro:property name="tableheight" value="0.78" />
-  <xacro:property name="tablewidth" value="1.00" />
-  <xacro:property name="tabledepth" value="0.80" />
-  <xacro:property name="tabletag_size" value="0.20" />
   <material name="black">
     <color rgba="0.0 0.0 0.0 1.0"/>
@@ -198,36 +193,4 @@
     <kd>1.0</kd>
   </gazebo>
-  <link name="table">
-    <inertial>
-      <origin xyz="0 0 ${tableheight/2}" />
-      <mass value="10" />
-      <inertia  ixx="1" ixy="0" ixz="0" iyy="1" iyz="0" izz="1" />
-    </inertial>
-    <visual>
-      <material name="brown" />
-      <origin xyz="0 0 ${tableheight/2}" />
-      <geometry>
-        <box size="0.80 1.0 ${tableheight}" />
-      </geometry>
-    </visual>
-    <collision>
-      <origin xyz="0 0 ${tableheight/2}" />
-      <geometry>
-        <box size="0.80 1.0 ${tableheight}" />
-      </geometry>
-    </collision>
-  </link>
-  <gazebo reference="table">
-    <material>Gazebo/Blue</material>
-    <turnGravityOff>false</turnGravityOff>
-    <selfCollide>true</selfCollide>
-    <!-- kp: stiffness kd: damping mu1, mu2: friction -->
-    <mu1>100.0</mu1>
-    <mu2>100.0</mu2>
-    <kp>1000000.0</kp>
-    <kd>1.0</kd>
-  </gazebo>
-  <link name="table_top"/>
-  <link name="table_tag"/>
   <link name="shelf">
     <inertial>
@@ -349,29 +312,4 @@
     <child link="cable_duct"/>
     <origin xyz="0.475 -0.135 ${roomheight/2}" rpy="0 0 0" />
-  </joint>
-  <xacro:unless value="$(arg floating_table)">
-  <joint name="table_joint" type="fixed">
-    <parent link="floor"/>
-    <child link="table"/>
-    <!-- actual wall is 2.5cm further back from table, but is modelled at the position of the small ur5 adapter plate -->
-   <!-- <origin xyz="0.73 0.30 0" rpy="0 0 0" /> -->
-    <origin xyz="0.89 0.74 0" rpy="0 0 0" />
-  </joint>
-  </xacro:unless>
-  <xacro:if value="$(arg floating_table)">
-  <joint name="table_joint" type="floating">
-    <parent link="floor"/>
-    <child link="table"/>
-  </joint>
-  </xacro:if>
-  <joint name="table_top_joint" type="fixed">
-    <parent link="table"/>
-    <child link="table_top"/>
-    <origin xyz="0 0 ${tableheight}" rpy="0 0 0"/>
-  </joint>
-  <joint name="table_tag_joint" type="fixed">
-    <parent link="table_top"/>
-    <child link="table_tag"/>
-    <origin xyz="${tabledepth/2-tabletag_size/2} ${tablewidth/2-tabletag_size/2} 0" rpy="0 0 ${pi}"/>
   </joint>
   <joint name="shelf_joint" type="fixed">

File: tams_ur5_setup_description/urdf/tams_ur5_setup.urdf.xacro (robot description, xacro)
@@ -6,4 +6,6 @@
   <!-- arm -->
   <xacro:include filename="$(find tams_ur5_description)/urdf/arm.urdf.xacro" />
+  <!-- table -->
+  <xacro:include filename="$(find tams_ur5_setup_description)/urdf/table.urdf.xacro" />
   <link name="world" />
   <joint name="world_floor_joint" type="fixed">
@@ -23,3 +25,10 @@
     <origin xyz="0 0 0.003" rpy="0.0 0.0 ${pi/2}" />
   </joint>
+  <joint name="table_joint" type="fixed">
+    <parent link="floor"/>
+    <child link="table"/>
+    <!-- actual wall is 2.5cm further back from table, but is modelled at the position of the small ur5 adapter plate -->
+   <!-- <origin xyz="0.73 0.30 0" rpy="0 0 0" /> -->
+    <origin xyz="0.89 0.74 0" rpy="0 0 0" />
+  </joint>
 </robot>
