Commit message: actually *use* table dimensions...

File: tams_ur5_setup_description/urdf/table.urdf.xacro (robot description, xacro)
@@ -16,5 +16,5 @@
       <origin xyz="0 0 ${tableheight/2}" />
       <geometry>
-        <box size="0.80 1.0 ${tableheight}" />
+        <box size="${tabledepth} ${tablewidth} ${tableheight}" />
       </geometry>
     </visual>
@@ -22,5 +22,5 @@
       <origin xyz="0 0 ${tableheight/2}" />
       <geometry>
-        <box size="0.80 1.0 ${tableheight}" />
+        <box size="${tabledepth} ${tablewidth} ${tableheight}" />
       </geometry>
     </collision>

Commit message: adjust values for mtc_pour experiments

File: tams_ur5_setup_description/urdf/table.urdf.xacro (robot description, xacro)
@@ -3,5 +3,5 @@
        name="tams_ur5_table" >
   <xacro:property name="tableheight" value="0.78" />
-  <xacro:property name="tablewidth" value="1.00" />
+  <xacro:property name="tablewidth" value="1.50" />
   <xacro:property name="tabledepth" value="0.80" />
   <xacro:property name="tabletag_size" value="0.20" />
