Commit message: fix deprecation warning Using load_yaml() directly is deprecated. Use xacro.load_yaml() instead.

File: tams_ur5_description/urdf/ur5.urdf.xacro (robot description, xacro)
@@ -19,5 +19,5 @@
   <!-- Loads the joint ranges configuration of the ur5 -->
   <xacro:arg name="joint_ranges_config" default="$(find tams_ur5_description)/config/joint_ranges/default.yaml" />
-  <xacro:property name="joint_limits" value="${load_yaml('$(arg joint_ranges_config)')}"/>
+  <xacro:property name="joint_limits" value="${xacro.load_yaml('$(arg joint_ranges_config)')}"/>
   <!-- Kinematic model -->
   <!-- Properties from urcontrol.conf -->
