Commit message: simplify tams_ur5 launch file name and xacro details

File: tams_ur5_description/urdf/arm.urdf.xacro (robot description, xacro)
@@ -2,5 +2,4 @@
 <robot xmlns:xacro="http://www.ros.org/wiki/xacro"
        name="arm" >
-  <xacro:arg name="r200" default="false" />
   <!-- include macro definitions -->
   <xacro:include filename="$(find tams_ur5_description)/urdf/ur5.urdf.xacro" />
@@ -10,5 +9,4 @@
   <xacro:include filename="$(find tams_ur5_description)/urdf/s_model_adapter.urdf.xacro" />
   <xacro:include filename="$(find tams_ur5_description)/urdf/plug_collision_model.urdf.xacro" />
-  <xacro:include filename="$(find tams_ur5_description)/urdf/mounted_camera.urdf.xacro" />
   <!-- arm -->
   <!-- xamla_cap is a custom parameter in TAMS' fork of the universal_robot repository,
@@ -19,10 +17,4 @@
     <origin xyz="0.0045 0.0 0.0" rpy="0.0 ${pi/2} 0.0" />
   </xacro:ft_adapter>
-  <!-- mounted_camera -->
-  <xacro:if value="$(arg r200)">
-    <xacro:mounted_camera name="mounted_camera" parent="ft_adapter">
-        <origin xyz="0 0 0.0" rpy="0 0 0" />
-    </xacro:mounted_camera>
-  </xacro:if>
   <!-- ft150 -->
   <xacro:robotiq_fts150 prefix="ft_" parent="ur5_ee_link">
