Commit message: add collision object for USB hub

File: tams_ur5_description/urdf/plug_collision_model.urdf.xacro (robot description, xacro)
@@ -47,4 +47,26 @@
       <parent link="${parent}"/>
     </joint>
+    <!-- usb hub -->
+    <link name="${name}_link_3">
+      <!-- TODO values for inertial are not correct -->
+      <inertial>
+        <mass value="0.2" />
+        <origin xyz="0.0 0.0 0.0" />
+        <inertia ixx="0.002708332" ixy="0.0" ixz="0.0"
+                 iyy="0.000708333" iyz="0.0"
+                 izz="0.003333332" />
+      </inertial>
+      <collision>
+        <origin xyz="0.025 -0.0 0.06" rpy="0.0 0.0 0.0" />
+        <geometry>
+          <box size="0.08 0.15 0.13"/>
+        </geometry>
+      </collision>
+    </link>
+    <joint name="${name}_link_3_joint" type="fixed">
+      <xacro:insert_block name="origin" />
+      <child link="${name}_link_3" />
+      <parent link="${parent}"/>
+    </joint>
   </xacro:macro>
 </robot>

Commit message: add visuals for cable boxes
Otherwise collisions are not correctly visualized in RViz with the
MotionPlanning panel.

File: tams_ur5_description/urdf/plug_collision_model.urdf.xacro (robot description, xacro)
@@ -13,4 +13,13 @@
                  izz="0.003333332" />
       </inertial>
+      <visual>
+        <origin xyz="0.08 -0.05 0.0" rpy="0.0 0.0 0.0" />
+        <geometry>
+          <box size="0.08 0.10 0.075"/>
+        </geometry>
+        <material name="${name}_link1_mat">
+          <color rgba="0.7 0.7 0.7 0.3"/>
+        </material>
+      </visual>
       <collision>
         <origin xyz="0.08 -0.05 0.0" rpy="0.0 0.0 0.0" />
@@ -35,4 +44,13 @@
                  izz="0.003333332" />
       </inertial>
+      <visual>
+        <origin xyz="0.025 -0.025 0.06" rpy="0.0 0.0 0.0" />
+        <geometry>
+          <box size="0.03 0.09 0.12"/>
+        </geometry>
+        <material name="${name}_link2_mat">
+          <color rgba="0.7 0.7 0.7 0.3"/>
+        </material>
+      </visual>
       <collision>
         <origin xyz="0.025 -0.025 0.06" rpy="0.0 0.0 0.0" />
@@ -57,4 +75,13 @@
                  izz="0.003333332" />
       </inertial>
+      <visual>
+        <origin xyz="0.025 -0.0 0.06" rpy="0.0 0.0 0.0" />
+        <geometry>
+          <box size="0.08 0.15 0.13"/>
+        </geometry>
+        <material name="${name}_link3_mat">
+          <color rgba="0.7 0.7 0.7 0.3"/>
+        </material>
+      </visual>
       <collision>
         <origin xyz="0.025 -0.0 0.06" rpy="0.0 0.0 0.0" />
